File: Hardware Notes/PCB Design/123-pcb-design.kicad_pcb (KiCad board)
At the start: 2 copper layers, 2 parts, among them U1 MCP73871, U3 HX711

Commit message: updated to v1 circuit
Parts:
- added U1: ESP32-C3-MINI-1, PCM_Espressif:ESP32-C3-MINI-1, F.Cu at (152.4, 51.6)
- moved U2 8.74 mm to (148.5, 64.0)
- moved U3 8.08 mm to (155.5, 66.0)
- renumbered U1 to U2
Connections:
- U2 pad 1: Net-(U2-IO6) -> VSUP
- U2 pad 20: Net-(U2-IO6) -> VSUP

Commit message: pcb rev2 and routing complete
Parts:
- added C1: 0.1μF, Capacitor_SMD:C_0402_1005Metric, F.Cu at (156.0, 92.5)
- added C2: 10μF, Capacitor_SMD:C_0402_1005Metric, F.Cu at (150.5, 92.5)
- added C3: 0.1μF, Capacitor_SMD:C_0402_1005Metric, F.Cu at (157.0, 84.0)
- added C4: 0.1μF, Capacitor_SMD:C_0402_1005Metric, F.Cu at (153.5, 79.5)
- added C5: 4.7μF, Capacitor_SMD:C_0603_1608Metric, F.Cu at (144.0, 65.5)
- added C6: 4.7μF, Capacitor_SMD:C_0603_1608Metric, F.Cu at (144.1, 72.1)
- added C7: 4.7μF, Capacitor_SMD:C_0603_1608Metric, F.Cu at (144.1, 79.6)
- added C8: 4.7μF, Capacitor_SMD:C_0603_1608Metric, F.Cu at (144.1, 82.6)
- added J1: JST 1x02, Connector_JST:JST_EH_S2B-EH_1x02_P2.50mm_Horizontal, F.Cu at (140.0, 90.8)
- added J2: JST 1x02, Connector_JST:JST_EH_S2B-EH_1x02_P2.50mm_Horizontal, F.Cu at (140.0, 82.2)
- added J3: JST 1x04, Connector_JST:JST_EH_S4B-EH_1x04_P2.50mm_Horizontal, F.Cu at (162.5, 84.2)
- added L1: 3.3μH, Inductor_SMD:L_0402_1005Metric, F.Cu at (150.5, 87.0)
- added R1: 20k, Resistor_SMD:R_0402_1005Metric_Pad0.72x0.64mm_HandSolder, F.Cu at (152.5, 84.0)
- added R2: 20k, Resistor_SMD:R_0402_1005Metric_Pad0.72x0.64mm_HandSolder, F.Cu at (154.5, 88.0)
- added R3: 100, Resistor_SMD:R_0402_1005Metric_Pad0.72x0.64mm_HandSolder, F.Cu at (159.0, 86.0)
- added R4: 100, Resistor_SMD:R_0402_1005Metric_Pad0.72x0.64mm_HandSolder, F.Cu at (159.0, 82.5)
- added R5: 0, Resistor_SMD:R_0402_1005Metric_Pad0.72x0.64mm_HandSolder, F.Cu at (144.0, 76.1)
- moved U2 10.4 mm to (138.1, 62.9), turned to 180 degrees
- moved U3 8.54 mm to (152.5, 74.0), turned to 90 degrees
Connections:
- net E- renamed GND
- U2 pad : (no net) -> U2-J1_NEG
- U2 pad 14: Net-(BAT1-+) -> Net-(U2-V_{BAT}-Pad14)
- U2 pad 15: Net-(BAT1-+) -> U2-V_{BAT}-Pad15
- U2 pad 16: unconnected-(U1-V_{BAT_SENSE}-Pad16) -> Net-(U2-V_{BAT_SENSE})
- U2 pad 18: Net-(J1-CC1) -> U2-J1_POS
Routing:
- net GND: track 0.00 -> 139.1 mm
- net VSUP: track 0.00 -> 35.1 mm
- net Net-(U3-AVDD): track 0.00 -> 29.8 mm
- net U2-J1_POS: track 0.00 -> 26.9 mm, vias 0 -> 1
- net U2-J1_NEG: track 0.00 -> 25.2 mm, vias 0 -> 1
- net Net-(U2-V_{BAT}-Pad14): track 0.00 -> 24.7 mm
- net U2-V_{BAT}-Pad15: track 0.00 -> 22.6 mm
- net Net-(U3-INA-): track 0.00 -> 13.8 mm
- net Net-(U2-V_{BAT_SENSE}): track 0.00 -> 13.5 mm
- net GPIO_5/ADC_2: track 0.00 -> 12.9 mm
- net GPIO_4/ADC_1: track 0.00 -> 12.7 mm
- net Net-(U3-INA+): track 0.00 -> 12.5 mm
- net Net-(U3-VFB): track 0.00 -> 12.4 mm
- net Net-(U3-VBG): track 0.00 -> 3.20 mm

Commit message: board rev3
Parts:
- moved U2 9.25 mm to (137.9, 72.1)
- moved U1 8.94 mm to (152.5, 60.5)
- moved C5 6.50 mm to (144.0, 72.0)
- moved C6 1.90 mm to (144.1, 74.0)
Connections:
- U2 pad 10: Net-(U2-V_{SS}-Pad10) -> GND
- U2 pad 11: Net-(U2-V_{SS}-Pad10) -> GND
- U2 pad 21: Net-(U2-V_{SS}-Pad10) -> GND
Routing:
- net GND: track 139.1 -> 0.03 mm
- net U2-J1_NEG: track 25.2 -> 14.9 mm
- net VSUP: track 35.1 -> 25.2 mm
- net U2-J1_POS: track 26.9 -> 17.6 mm
- net Net-(U2-V_{BAT}-Pad14): track 24.7 -> 15.6 mm
- net GPIO_4/ADC_1: track 12.7 -> 3.68 mm
- net GPIO_5/ADC_2: track 12.9 -> 3.87 mm
- net U2-V_{BAT}-Pad15: track 22.6 -> 14.9 mm
- net Net-(U2-V_{BAT_SENSE}): track 13.5 -> 11.3 mm
- added copper zone on B.Cu, net GND
- added copper zone on F.Cu, net GND
