File: Hardware Notes/PCB Design/123-pcb-design.kicad_sch (KiCad schematic)
At the start: 21 parts, among them J3 Conn_01x04_Pin, U1 ESP32-C3-MINI-1, U2 MCP73871, U3 HX711

Commit message: pcb rev 4 w/ battery monitor circuit
Parts:
- added R5, R6: 1k, symbol Device:R_Small_US
Connections:
- net GND: now also R6.2
- net VSUP: now also R5.2
- net at U1.5 (GPIO2/ADC1_CH2): now also R5.1, R6.1
Other:
- note added: "Battery Measurement"

Commit message: DRC passes for schematic
Parts:
- removed 4.9: 4.7μF, symbol Device:C_Small
- R5, R6: value 1k -> 100k
- U2: footprint Package_DFN_QFN:QFN-20-1EP_4x4mm_P0.5mm_EP2.5x2.5mm -> Package_DFN_QFN:VQFN-28-1EP_5x5mm_P0.5mm_EP3.25x3.25mm
Connections:
- net at 4.3.1, 4.8.1, J2.1 (Pin_1)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: no longer U2.16 (V_{BAT_SENSE})
Changed lines of the file:
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@@
 	)
 	(junction
-		(at 101.6 143.51)
-		(diameter 0)
-		(color 0 0 0 0)
-	)
-	(junction
 		(at 107.95 46.99)
 		(diameter 0)
@@
 	)
 	(junction
-		(at 101.6 138.43)
-		(diameter 0)
-		(color 0 0 0 0)
-	)
-	(junction
 		(at 49.53 114.3)
 		(diameter 0)
@@
 	(wire
 		(pts
-			(xy 101.6 151.13) (xy 110.49 151.13)
-		)
-		(stroke
-			(width 0)
-			(type default)
-		)
-	)
-	(wire
-		(pts
 			(xy 226.06 55.88) (xy 215.9 55.88)
 		)
@@
 	(wire
 		(pts
-			(xy 95.25 138.43) (xy 101.6 138.43)
-		)
-		(stroke
-			(width 0)
-			(type default)
-		)
-	)
-	(wire
-		(pts
 			(xy 62.23 27.94) (xy 64.77 27.94)
 		)
@@
 	(wire
 		(pts
-			(xy 101.6 143.51) (xy 101.6 151.13)
-		)
-		(stroke
-			(width 0)
-			(type default)
-		)
-	)
-	(wire
-		(pts
 			(xy 107.95 115.57) (xy 109.22 115.57)
 		)
@@
 	(wire
 		(pts
-			(xy 101.6 138.43) (xy 115.57 138.43)
+			(xy 95.25 138.43) (xy 115.57 138.43)
 		)
 		(stroke
@@
 	(wire
 		(pts
-			(xy 95.25 143.51) (xy 101.6 143.51)
-		)
-		(stroke
-			(width 0)
-			(type default)
-		)
-	)
-	(wire
-		(pts
 			(xy 200.66 39.37) (xy 232.41 39.37)
 		)
@@
 	(wire
 		(pts
-			(xy 101.6 143.51) (xy 101.6 138.43)
-		)
-		(stroke
-			(width 0)
-			(type default)
-		)
-	)
-	(wire
-		(pts
 			(xy 115.57 138.43) (xy 115.57 151.13)
 		)
@@
 	(symbol
 		(lib_id "power:GND")
-		(at 110.49 156.21 0)
-		(unit 1)
-		(body_style 1)
-		(exclude_from_sim no)
-		(in_bom yes)
-		(on_board yes)
-		(in_pos_files yes)
-		(dnp no)
-		(fields_autoplaced yes)
-		(property "Reference" "#PWR011"
-			(at 110.49 162.56 0)
-			(hide yes)
-			(show_name no)
-			(do_not_autoplace no)
-			(effects
-				(font
-					(size 1.27 1.27)
-				)
-			)
-		)
-		(property "Value" "GND"
-			(at 110.49 161.29 0)
-			(show_name no)
-			(do_not_autoplace no)
-			(effects
-				(font
-					(size 1.27 1.27)
-				)
-			)
-		)
-		(property "Footprint" ""
-			(at 110.49 156.21 0)
-			(hide yes)
-			(show_name no)
-			(do_not_autoplace no)
-			(effects
-				(font
-					(size 1.27 1.27)
-				)
-			)
-		)
-		(property "Datasheet" ""
-			(at 110.49 156.21 0)
-			(hide yes)
-			(show_name no)
-			(do_not_autoplace no)
-			(effects
-				(font
-					(size 1.27 1.27)
-				)
-			)
-		)
-		(property "Description" "Power symbol creates a global label with name \"GND\" , ground"
-			(at 110.49 156.21 0)
-			(hide yes)
-			(show_name no)
-			(do_not_autoplace no)
-			(effects
-				(font
-					(size 1.27 1.27)
-				)
-			)
-		)
-		(pin "1"
-		)
-		(instances
-			(project "123-pcb-design"
-				(path "/59495f75-6f35-499b-95d0-e7e9548b242d"
-					(reference "#PWR011")
-					(unit 1)
-				)
-			)
-		)
-	)
-	(symbol
-		(lib_id "power:GND")
 		(at 233.68 97.79 0)
 		(unit 1)
@@
 			)
 		)
-		(property "Value" "1k"
+		(property "Value" "100k"
 			(at 115.57 49.022 90)
 			(show_name no)
@@
 			)
 		)
-		(property "Value" "1k"
-			(at 110.49 52.832 0)
+		(property "Value" "100k"
+			(at 111.506 52.832 0)
 			(show_name no)
 			(do_not_autoplace no)
@@
 			)
 		)
-		(property "Footprint" "Package_DFN_QFN:QFN-20-1EP_4x4mm_P0.5mm_EP2.5x2.5mm"
+		(property "Footprint" "Package_DFN_QFN:VQFN-28-1EP_5x5mm_P0.5mm_EP3.25x3.25mm"
 			(at 82.55 168.91 0)
 			(hide yes)
@@
 					(unit 1)
 				)
-			)
-		)
-	)
-	(symbol
-		(lib_id "Device:C_Small")
-		(at 110.49 153.67 0)
-		(unit 1)
-		(body_style 1)
-		(exclude_from_sim no)
-		(in_bom yes)
-		(on_board yes)
-		(in_pos_files yes)
-		(dnp no)
-		(property "Reference" "4.9"
-			(at 113.03 152.4062 0)
-			(hide yes)
-			(show_name no)
-			(do_not_autoplace no)
-			(effects
-				(font
-					(size 1.27 1.27)
-				)
-				(justify left)
-			)
-		)
-		(property "Value" "4.7μF"
-			(at 113.03 153.67 0)
-			(show_name no)
-			(do_not_autoplace no)
-			(effects
-				(font
-					(size 1.27 1.27)
-				)
-				(justify left)
-			)
-		)
-		(property "Footprint" ""
-			(at 110.49 153.67 0)
-			(hide yes)
-			(show_name no)
-			(do_not_autoplace no)
-			(effects
-				(font
-					(size 1.27 1.27)
-				)
-			)
-		)
-		(property "Datasheet" ""
-			(at 110.49 153.67 0)
-			(hide yes)
-			(show_name no)
-			(do_not_autoplace no)
-			(effects
-				(font
-					(size 1.27 1.27)
-				)
-			)
-		)
-		(property "Description" "Unpolarized capacitor, small symbol"
-			(at 110.49 153.67 0)
-			(hide yes)
-			(show_name no)
-			(do_not_autoplace no)
-			(effects
-				(font
-					(size 1.27 1.27)
-				)
-			)
-		)
-		(pin "1"
-		)
-		(pin "2"
-		)
-		(instances
-			(project "123-pcb-design"
-				(path "/59495f75-6f35-499b-95d0-e7e9548b242d"
-					(reference "4.9")
-					(unit 1)
-				)

Commit message: new pcb documents, references added to schematic
Parts:
- renumbered 4.4 to C1, 4.5 to C2, 4.6 to C4, 4.2 to C5, 4.3 to C6, 4.8 to C7, 4.10 to C8, 4.11 to C9, R4 to R3, R3 to R4
Changed lines of the file:
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@@
 	(text "Battery Measurement"
 		(exclude_from_sim no)
-		(at 116.586 44.196 0)
+		(at 116.586 43.18 0)
 		(effects
 			(font
@@
 	)
 	(junction
-		(at 193.04 62.23)
+		(at 215.9 55.88)
 		(diameter 0)
 		(color 0 0 0 0)
 	)
 	(junction
-		(at 215.9 55.88)
+		(at 182.88 30.48)
 		(diameter 0)
 		(color 0 0 0 0)
@@
 	)
 	(junction
-		(at 182.88 30.48)
+		(at 120.65 151.13)
 		(diameter 0)
 		(color 0 0 0 0)
 	)
 	(junction
-		(at 49.53 114.3)
+		(at 46.99 114.3)
 		(diameter 0)
 		(color 0 0 0 0)
 	)
 	(junction
-		(at 120.65 151.13)
+		(at 193.04 62.23)
 		(diameter 0)
 		(color 0 0 0 0)
@@
 	(wire
 		(pts
-			(xy 49.53 114.3) (xy 55.88 114.3)
+			(xy 217.17 62.23) (xy 217.17 67.31)
 		)
 		(stroke
@@
 	(wire
 		(pts
-			(xy 217.17 62.23) (xy 217.17 67.31)
+			(xy 232.41 49.53) (xy 226.06 49.53)
 		)
 		(stroke
@@
 	(wire
 		(pts
-			(xy 232.41 49.53) (xy 226.06 49.53)
+			(xy 107.95 46.99) (xy 100.33 46.99)
 		)
 		(stroke
@@
 	(wire
 		(pts
-			(xy 107.95 46.99) (xy 100.33 46.99)
+			(xy 46.99 114.3) (xy 55.88 114.3)
 		)
 		(stroke
@@
 	(wire
 		(pts
-			(xy 38.1 114.3) (xy 49.53 114.3)
+			(xy 38.1 114.3) (xy 46.99 114.3)
 		)
 		(stroke
@@
 		(in_pos_files yes)
 		(dnp no)
-		(property "Reference" "4.11"
+		(property "Reference" "C9"
 			(at 62.23 113.0362 0)
-			(hide yes)
 			(show_name no)
 			(do_not_autoplace no)
@@
 		)
 		(property "Value" "10μF"
-			(at 62.23 114.3 0)
+			(at 62.23 115.062 0)
 			(show_name no)
 			(do_not_autoplace no)
@@
 			(project "123-pcb-design"
 				(path "/59495f75-6f35-499b-95d0-e7e9548b242d"
-					(reference "4.11")
+					(reference "C9")
 					(unit 1)
 				)
@@
 		(in_pos_files yes)
 		(dnp no)
-		(fields_autoplaced yes)
 		(property "Reference" "R1"
-			(at 203.2 33.0199 0)
-			(hide yes)
+			(at 202.438 33.528 0)
 			(show_name no)
 			(do_not_autoplace no)
@@
 		)
 		(property "Value" "20k"
-			(at 203.2 34.2899 0)
+			(at 202.438 35.306 0)
 			(show_name no)
 			(do_not_autoplace no)
@@
 		(property "Reference" "L1"
 			(at 191.77 25.4 90)
-			(hide yes)
 			(show_name no)
 			(do_not_autoplace no)
@@
 		(in_pos_files yes)
 		(dnp no)
-		(property "Reference" "4.8"
-			(at 123.19 152.4062 0)
-			(hide yes)
+		(property "Reference" "C7"
+			(at 123.19 152.654 0)
 			(show_name no)
 			(do_not_autoplace no)
@@
 		)
 		(property "Value" "4.7μF"
-			(at 123.19 153.67 0)
+			(at 123.19 154.686 0)
 			(show_name no)
 			(do_not_autoplace no)
@@
 			(project "123-pcb-design"
 				(path "/59495f75-6f35-499b-95d0-e7e9548b242d"
-					(reference "4.8")
+					(reference "C7")
 					(unit 1)
 				)
@@
 		(in_pos_files yes)
 		(dnp no)
-		(property "Reference" "4.6"
-			(at 207.01 63.5062 0)
-			(hide yes)
+		(property "Reference" "C4"
+			(at 207.01 63.754 0)
 			(show_name no)
 			(do_not_autoplace no)
@@
 		)
 		(property "Value" "0.1μF"
-			(at 207.01 64.77 0)
+			(at 207.01 65.786 0)
 			(show_name no)
 			(do_not_autoplace no)
@@
 			(project "123-pcb-design"
 				(path "/59495f75-6f35-499b-95d0-e7e9548b242d"
-					(reference "4.6")
+					(reference "C4")
 					(unit 1)
 				)
@@
 		(in_pos_files yes)
 		(dnp no)
-		(property "Reference" "4.3"
-			(at 123.19 139.7062 0)
-			(hide yes)
+		(property "Reference" "C6"
+			(at 123.19 139.954 0)
 			(show_name no)
 			(do_not_autoplace no)
@@
 		)
 		(property "Value" "4.7μF"
-			(at 123.19 140.97 0)
+			(at 123.19 142.24 0)
 			(show_name no)
 			(do_not_autoplace no)
@@
 			(project "123-pcb-design"
 				(path "/59495f75-6f35-499b-95d0-e7e9548b242d"
-					(reference "4.3")
+					(reference "C6")
 					(unit 1)
 				)
@@
 		(dnp no)
 		(property "Reference" "R5"
-			(at 114.2999 44.45 0)
-			(hide yes)
+			(at 116.84 44.958 90)
 			(show_name no)
 			(do_not_autoplace no)
@@
 	(symbol
 		(lib_id "power:GND")
-		(at 49.53 119.38 0)
+		(at 46.99 119.38 0)
 		(unit 1)
 		(body_style 1)
@@
 		(fields_autoplaced yes)
 		(property "Reference" "#PWR012"
-			(at 49.53 125.73 0)
+			(at 46.99 125.73 0)
 			(hide yes)
 			(show_name no)
@@
 		)
 		(property "Value" "GND"
-			(at 49.53 124.46 0)
+			(at 46.99 124.46 0)
 			(show_name no)
 			(do_not_autoplace no)
@@
 		)
 		(property "Footprint" ""
-			(at 49.53 119.38 0)
+			(at 46.99 119.38 0)
 			(hide yes)
 			(show_name no)
@@
 		)
 		(property "Datasheet" ""
-			(at 49.53 119.38 0)
+			(at 46.99 119.38 0)
 			(hide yes)
 			(show_name no)
@@
 		)
 		(property "Description" "Power symbol creates a global label with name \"GND\" , ground"
-			(at 49.53 119.38 0)
+			(at 46.99 119.38 0)
 			(hide yes)
 			(show_name no)
@@
 		(dnp no)
 		(property "Reference" "R6"
-			(at 110.49 52.0699 0)
-			(hide yes)
+			(at 109.22 52.07 0)
 			(show_name no)
 			(do_not_autoplace no)
@@
 		)
 		(property "Value" "100k"
-			(at 111.506 52.832 0)
+			(at 111.506 54.102 0)
 			(show_name no)
 			(do_not_autoplace no)
@@
 		(in_pos_files yes)
 		(dnp no)
-		(property "Reference" "4.2"
-			(at 111.76 120.6562 0)
-			(hide yes)
+		(property "Reference" "C5"
+			(at 111.76 121.158 0)
 			(show_name no)
 			(do_not_autoplace no)
@@
 		)
 		(property "Value" "4.7μF"
-			(at 111.76 121.92 0)
+			(at 111.76 123.4378 0)
 			(show_name no)
 			(do_not_autoplace no)
@@
 			(project "123-pcb-design"
 				(path "/59495f75-6f35-499b-95d0-e7e9548b242d"
-					(reference "4.2")
+					(reference "C5")
 					(unit 1)
 				)
@@
 		(in_pos_files yes)
 		(dnp no)
-		(property "Reference" "4.4"
-			(at 175.26 31.7562 0)
-			(hide yes)
+		(property "Reference" "C1"
+			(at 175.26 32.512 0)
 			(show_name no)
 			(do_not_autoplace no)
@@
 		)
 		(property "Value" "0.1μF"
-			(at 175.26 33.02 0)
+			(at 175.006 34.544 0)
 			(show_name no)
 			(do_not_autoplace no)
@@
 			(project "123-pcb-design"
 				(path "/59495f75-6f35-499b-95d0-e7e9548b242d"
-					(reference "4.4")
+					(reference "C1")
 					(unit 1)
 				)
@@
 	(symbol
 		(lib_id "Device:C_Small")
-		(at 49.53 116.84 0)
+		(at 46.99 116.84 0)
 		(unit 1)
 		(body_style 1)
@@
 		(in_pos_files yes)
 		(dnp no)
-		(property "Reference" "4.10"
-			(at 52.07 115.5762 0)
-			(hide yes)
+		(property "Reference" "C8"
+			(at 49.53 115.5762 0)
 			(show_name no)
 			(do_not_autoplace no)
@@
 		)
 		(property "Value" "10μF"
-			(at 52.07 116.84 0)
+			(at 49.53 117.602 0)
 			(show_name no)
 			(do_not_autoplace no)
@@
 		)
 		(property "Footprint" ""
-			(at 49.53 116.84 0)
+			(at 46.99 116.84 0)
 			(hide yes)
 			(show_name no)
@@
 		)
 		(property "Datasheet" ""
-			(at 49.53 116.84 0)
+			(at 46.99 116.84 0)
 			(hide yes)
 			(show_name no)
@@
 		)
 		(property "Description" "Unpolarized capacitor, small symbol"
-			(at 49.53 116.84 0)
+			(at 46.99 116.84 0)
 			(hide yes)
 			(show_name no)
@@
 			(project "123-pcb-design"
 				(path "/59495f75-6f35-499b-95d0-e7e9548b242d"
-					(reference "4.10")
+					(reference "C8")
 					(unit 1)
 				)
@@
 		(in_pos_files yes)
 		(dnp no)
-		(property "Reference" "R4"
-			(at 209.5499 53.34 0)
-			(hide yes)
+		(property "Reference" "R3"
+			(at 211.836 53.34 90)
 			(show_name no)
 			(do_not_autoplace no)
@@
 			(project "123-pcb-design"
 				(path "/59495f75-6f35-499b-95d0-e7e9548b242d"
-					(reference "R4")
+					(reference "R3")
 					(unit 1)
 				)
@@
 		(in_pos_files yes)
 		(dnp no)
-		(property "Reference" "R3"
-			(at 209.5499 43.18 0)
-			(hide yes)
+		(property "Reference" "R4"
+			(at 212.09 48.006 90)
 			(show_name no)
 			(do_not_autoplace no)
@@
 			(project "123-pcb-design"
 				(path "/59495f75-6f35-499b-95d0-e7e9548b242d"
-					(reference "R3")
+					(reference "R4")
 					(unit 1)
 				)
@@
 		(in_pos_files yes)
 		(dnp no)
-		(fields_autoplaced yes)
 		(property "Reference" "R2"
-			(at 195.58 48.2599 0)
-			(hide yes)
+			(at 195.072 49.022 0)
 			(show_name no)
 			(do_not_autoplace no)
@@
 		)
 		(property "Value" "8.2k"
-			(at 195.58 49.5299 0)
+			(at 195.072 50.8 0)
 			(show_name no)
 			(do_not_autoplace no)
@@
 		(in_pos_files yes)
 		(dnp no)
-		(property "Reference" "4.5"
-			(at 185.42 31.7562 0)
-			(hide yes)
+		(property "Reference" "C2"
+			(at 185.674 32.766 0)
 			(show_name no)
 			(do_not_autoplace no)
@@
 		)
 		(property "Value" "10μF"
-			(at 185.42 33.02 0)
+			(at 185.166 34.544 0)
 			(show_name no)
 			(do_not_autoplace no)
@@
 			(project "123-pcb-design"
 				(path "/59495f75-6f35-499b-95d0-e7e9548b242d"
-					(reference "4.5")
+					(reference "C2")
 					(unit 1)
 				)
